File: demos/video/video.kicad_pcb (KiCad board)
At the start: 4 copper layers, 312 x 106.7 mm, 189 parts, among them J4 DB9FEM, P1 BNC, P10 CONN_1, P11 CONN_1, P12 CONN_1, P2 BNC, P3 BNC, P4 CONN_2, P5 CONN_5, P8 BNC, P9 CONN_1, Q1 BC848, Q2 BC848, Q3 BC848, U1 24C16, U10 BT812, U11 S5933_PQ160, U12 SIM4X32, U13 SIM4X32, U14 SIM4X32, U15 SIM4X32, U16 SIM4X32, U17 SIM4X32, U18 SIM4X32, U19 SIM4X32, U2 4C4001, U20 TDA8501, U21 XC1736APD8, U22 XC4003-VQ100, U23 XC4003/PQ100, U24 XC4005-PQ160, U3 74LS245, U4 74LS245, U5 74LS245, U6 74LS245, U7 AV9173, U8 BT253, U9 BT473, X1 10MHz, X2 30MHz, X3 4.433618MHz

Commit message: Update demos.
Routing:
- net GND: track 759.7 -> 758.5 mm
- net /graphic/VOSC: track 26.7 -> 25.9 mm
