File: demos/video/video.kicad_pcb (KiCad board)
At the start: 4 copper layers, 312 x 106.7 mm, 189 parts, among them J4 DB9FEM, P1 BNC, P10 CONN_1, P11 CONN_1, P12 CONN_1, P2 BNC, P3 BNC, P4 CONN_2, P5 CONN_5, P8 BNC, P9 CONN_1, Q1 BC848, Q2 BC848, Q3 BC848, U1 24C16, U10 BT812, U11 S5933_PQ160, U12 SIM4X32, U13 SIM4X32, U14 SIM4X32, U15 SIM4X32, U16 SIM4X32, U17 SIM4X32, U18 SIM4X32, U19 SIM4X32, U2 4C4001, U20 TDA8501, U21 XC1736APD8, U22 XC4003-VQ100, U23 XC4003/PQ100, U24 XC4005-PQ160, U3 74LS245, U4 74LS245, U5 74LS245, U6 74LS245, U7 AV9173, U8 BT253, U9 BT473, X1 10MHz, X2 30MHz, X3 4.433618MHz

Commit message: Update demos to V9 file formats except simulations.
Parts:
- C1, C10, C11, C12, C13, C14, C15, C16, C17, C18, C19, C2, C20, C21, C22, C23, C24, C25, C26, C27, C28, C29, C3, C30, C31, C32, C33, C34, C35, C36, C37, C38, C4, C43, C44, C45, C46, C47, C48, C5, C52, C53, C54, C58, C59, C6, C60, C61, C65, C66, C67, C68, C69, C7, C70, C71, C72, C73, C8, C9, R1, R10, R11, R12, R13, R14, R15, R16, R17, R18, R19, R2, R20, R21, R22, R23, R24, R25, R26, R27, R28, R29, R3, R30, R31, R32, R33, R34, R35, R36, R37, R38, R39, R4, R40, R41, R42, R43, R44, R45, R46, R47, R48, R5, R6, R7, R8, R9: footprint Resistor_SMD:R_1206_3216Metric_Pad1.30x1.75mm_HandSolder -> footprints:R_1206_3216Metric_Pad1.30x1.75mm_HandSolder
- C39, C40, C41, C42, C51, C55, C62, C63, C64: footprint Resistor_SMD:R_1210_3225Metric_Pad1.30x2.65mm_HandSolder -> footprints:R_1210_3225Metric_Pad1.30x2.65mm_HandSolder
- C49, C50: footprint Capacitor_THT:C_Disc_D3.0mm_W2.0mm_P2.50mm -> footprints:C_Disc_D3.0mm_W2.0mm_P2.50mm
- C56, C57: footprint Capacitor_Tantalum_SMD:CP_EIA-3528-21_Kemet-B_Pad1.50x2.35mm_HandSolder -> footprints:CP_EIA-3528-21_Kemet-B_Pad1.50x2.35mm_HandSolder
- J4: footprint Connector_Dsub:DSUB-9_Female_Horizontal_P2.77x2.84mm_EdgePinOffset14.56mm_Housed_MountingHolesOffset15.98mm -> footprints:DSUB-9_Female_Horizontal_P2.77x2.84mm_EdgePinOffset14.56mm_Housed_MountingHolesOffset15.98mm
- L1, L2, L3, L4, L5: footprint Resistor_SMD:R_1812_4532Metric_Pad1.30x3.40mm_HandSolder -> footprints:R_1812_4532Metric_Pad1.30x3.40mm_HandSolder
- P10, P11, P12, P9: footprint Connector_PinHeader_2.54mm:PinHeader_1x01_P2.54mm_Vertical -> footprints:PinHeader_1x01_P2.54mm_Vertical
- P4, W4, W5: footprint Connector_PinHeader_2.54mm:PinHeader_1x02_P2.54mm_Vertical -> footprints:PinHeader_1x02_P2.54mm_Vertical
- P5: footprint Connector_PinHeader_2.54mm:PinHeader_1x05_P2.54mm_Vertical -> footprints:PinHeader_1x05_P2.54mm_Vertical
- POT1: footprint Potentiometer_SMD:Potentiometer_Bourns_3314G_Vertical -> footprints:Potentiometer_Bourns_3314G_Vertical
- RR1, RR2, RR3, RR4, RR5, RR6, RR7, RR8: footprint Resistor_THT:R_Array_SIP9 -> footprints:R_Array_SIP9
- U1, U21: footprint Package_DIP:DIP-8_W7.62mm -> footprints:DIP-8_W7.62mm
- U10, U11, U24: footprint Package_QFP:PQFP-160_28x28mm_P0.65mm -> footprints:PQFP-160_28x28mm_P0.65mm
- U2: footprint Package_SO:SOIC-28W_7.5x17.9mm_P1.27mm -> footprints:SOIC-28W_7.5x17.9mm_P1.27mm
- U20: footprint Package_SO:SOIC-24W_7.5x15.4mm_P1.27mm -> footprints:SOIC-24W_7.5x15.4mm_P1.27mm
- U22: footprint Package_QFP:TQFP-100_14x14mm_P0.5mm -> footprints:TQFP-100_14x14mm_P0.5mm
- U23: footprint Package_QFP:PQFP-100_14x20mm_P0.65mm -> footprints:PQFP-100_14x20mm_P0.65mm
- U3, U4, U5, U6: footprint Package_SO:SOIC-20W_7.5x12.8mm_P1.27mm -> footprints:SOIC-20W_7.5x12.8mm_P1.27mm
- U7: footprint Package_SO:SSOP-8_3.95x5.21x3.27mm_P1.27mm -> footprints:SSOP-8_3.95x5.21x3.27mm_P1.27mm
- X1, X2: footprint Crystal:Crystal_HC18-U_Vertical -> footprints:Crystal_HC18-U_Vertical
- X3: footprint Crystal:Crystal_HC18-U_Horizontal -> footprints:Crystal_HC18-U_Horizontal
